Commit message: New world with properly working simulation of tb3, new simulation is based on repo: https://github.com/arshadlab/turtlebot3_multi_robot

File: urdf/turtlebot3_waffle.urdf (robot description, URDF)
Before this commit: robot turtlebot3_waffle, 13 links, 12 joints
Joints:
- joint camera_depth_joint: origin xyz=0.005 0.028 0.013 rpy=-1.57 0 -1.57 -> xyz=0.005 0.028 0.013 rpy=0 0 0
- joint camera_depth_optical_joint: origin xyz=0 0 0 rpy=0 0 0 -> xyz=0 0 0 rpy=-1.57 0 -1.57
